Commit message: URDF file for third arm

File: urdf/test_arm.urdf (robot description, URDF)
Before this commit: robot third_arm, 4 links, 3 joints
Links:
- added link extend_link1; visual box size=0.1 .26 .1
- added link extend_link2; visual box size=0.07 .20 .07
- added link finger1, mass 1; visual box size=0.01 .1 .02
- added link finger2, mass 1; visual box size=0.01 .1 .02
- added link gripper_motor, mass 1; visual cylinder length=0.07 radius=0.01
- added link lift_motor, mass 1; visual cylinder length=0.1 radius=0.05
- added link wrist_motor, mass 1; visual cylinder length=0.05 radius=0.03
- added link wrist_plate; visual box size=0.07 .02 .07
- link base_link: geometry visual cylinder length=0.6 radius=0.1
- link swivel_link: geometry visual box size=0.2 .15 .1
Joints:
- added joint extension: type prismatic, parent extend_link1, child extend_link2, origin xyz=0 0.07 0 rpy=0 0 0, axis 0 1 0, limit lower=0 upper=0.15 effort=10 velocity=5
- added joint finger1_to_gripper_motor: type revolute, parent gripper_motor, child finger1, origin xyz=0 0 0 rpy=0 0 0, axis 0 0 1, limit lower=0 upper=1 effort=5 velocity=0.5
- added joint finger2_to_gripper_motor: type revolute, parent gripper_motor, child finger2, origin xyz=0 0 0 rpy=0 0 0, axis 0 0 1, limit lower=-1 upper=0 effort=5 velocity=0.5, mimic joint=finger1_to_gripper_motor multiplier=-1
- added joint gripper_motor_to_plate: type fixed, parent wrist_plate, child gripper_motor, origin xyz=0 0.02 0 rpy=0 0 0
- added joint motor2_to_extend1: type fixed, parent lift_motor, child extend_link1, origin xyz=0 0.18 0 rpy=0 0 0
- added joint swivel_to_motor2: type revolute, parent swivel_link, child lift_motor, origin xyz=0 0.125 0 rpy=0 0 0, axis 1 0 0, limit lower=-1.5708 upper=1.5708 effort=10 velocity=0.314
- added joint wrist_motor_to_extension: type revolute, parent extend_link2, child wrist_motor, origin xyz=0 0.125 0 rpy=0 0 0, axis 0 1 0, limit lower=-1.5708 upper=1.5708 effort=5 velocity=0.5
- added joint wrist_motor_to_plate: type fixed, parent wrist_motor, child wrist_plate, origin xyz=0 0.035 0 rpy=0 0 0
- joint brace_block_link: origin xyz=0 -0.2 -0.2 rpy=0 0 0 -> xyz=0 -0.2 -0.15 rpy=0 0 0
- joint motor1_to_swivel_link: origin xyz=0 0.51 0 rpy=0 0 0 -> xyz=0 0.185 0 rpy=0 0 0
