Commit message: Combined WS computation

File: urdf/third_arm_human_old.urdf (robot description, URDF)
Before this commit: robot third_arm_with_human, 56 links, 55 joints
Links:
- link base_link: geometry visual cylinder length=0.3 radius=0.05
- link human/base: geometry visual cylinder length=-0.076637666482 radius=0.128063809513
- link human/head: geometry visual sphere radius=0.1
- link human/left_ankle: geometry visual box size=0.1 0.05 .005
- link human/left_elbow: geometry visual cylinder length=0.273206361701 radius=0.025
- link human/left_hip: geometry visual cylinder length=0.53151880807 radius=0.05
- link human/left_knee: geometry visual cylinder length=0.36903984413 radius=0.025
- link human/left_shoulder: geometry visual cylinder length=0.343212242182 radius=0.05
- link human/left_wrist: geometry visual box size=0.1 0.05 .005
- link human/neck: geometry visual cylinder length=0.198713359681 radius=0.04
- link human/right_ankle: geometry visual box size=0.1 0.05 .005
- link human/right_elbow: geometry visual cylinder length=0.273206361701 radius=0.025
- link human/right_hip: geometry visual cylinder length=0.53151880807 radius=0.05
- link human/right_knee: geometry visual cylinder length=0.36903984413 radius=0.025
- link human/right_shoulder: geometry visual cylinder length=0.343212242182 radius=0.05
- link human/right_wrist: geometry visual box size=0.1 0.05 .005
- link human/shoulder_center: geometry visual cylinder length=0.126849441152 radius=0.173623764208
- link human/spine: geometry visual cylinder length=0.262448400938 radius=0.153623764208
- link human/spine_0: geometry visual cylinder length=0.0900777328402 radius=0.133623764208
Joints:
- joint brace_block_link: origin xyz=0 -0.1 -0.05 rpy=0 0 0 -> xyz=0 -0.15 -0.05 rpy=0 0 0
- joint head: origin xyz=0 0 0.1 rpy=0 0 0 -> xyz=0 0 0.198713359681 rpy=0 0 0
- joint left_ankle_0: origin xyz=0.362 0 0 rpy=-1.57079632679 0 1.57079632679 -> xyz=0.36903984413 0 0 rpy=-1.57079632679 0 1.57079632679
- joint left_arm_mount: origin xyz=0 0.05 0.05 rpy=0 0 1.57079632679 -> xyz=0 0.173623764208 -0.00143826424372 rpy=0 0 1.57079632679
- joint left_elbow_0: origin xyz=0.406 0 0 rpy=0 0 0 -> xyz=0.343212242182 0 0 rpy=0 0 0
- joint left_foot: origin xyz=0.273 0 0 rpy=0 0 0 -> xyz=0.1 0 0 rpy=0 0 0
- joint left_hand: origin xyz=0.139 0 0 rpy=0 0 0 -> xyz=0.1 0 0 rpy=0 0 0
- joint left_hip_leg_mount: origin xyz=0 0.06 -0.018 rpy=0 1.57079632679 0 -> xyz=0 0.0780638095132 -0.076637666482 rpy=0 1.57079632679 0
- joint left_knee_0: origin xyz=0.469 0 0 rpy=1.57079632679 0 0 -> xyz=0.53151880807 0 0 rpy=1.57079632679 0 0
- joint left_wrist_0: origin xyz=0.417 0 0 rpy=0 0 0 -> xyz=0.273206361701 0 0 rpy=0 0 0
- joint neck_0: origin xyz=0 0 0.18 rpy=0 0 0 -> xyz=0 0 0.126849441152 rpy=0 0 0
- joint right_ankle_0: origin xyz=0.362 0 0 rpy=-1.57079632679 0 1.57079632679 -> xyz=0.36903984413 0 0 rpy=-1.57079632679 0 1.57079632679
- joint right_arm_mount: origin xyz=0 -0.05 0.05 rpy=0 0 -1.57079632679 -> xyz=0 -0.173623764208 -0.00143826424372 rpy=0 0 -1.57079632679
- joint right_elbow_0: origin xyz=0.406 0 0 rpy=0 0 0 -> xyz=0.343212242182 0 0 rpy=0 0 0
- joint right_foot: origin xyz=0.273 0 0 rpy=0 0 0 -> xyz=0.1 0 0 rpy=0 0 0
- joint right_hand: origin xyz=0.139 0 0 rpy=0 0 0 -> xyz=0.1 0 0 rpy=0 0 0
- joint right_hip_leg_mount: origin xyz=0 -0.06 -0.018 rpy=0 1.57079632679 0 -> xyz=0 -0.0780638095132 -0.076637666482 rpy=0 1.57079632679 0
- joint right_knee_0: origin xyz=0.469 0 0 rpy=1.57079632679 0 0 -> xyz=0.53151880807 0 0 rpy=1.57079632679 0 0
- joint right_wrist_0: origin xyz=0.417 0 0 rpy=0 0 0 -> xyz=0.273206361701 0 0 rpy=0 0 0
- joint shoulder_center: origin xyz=0 0 0.36 rpy=0 0 0 -> xyz=0 0 0.262448400938 rpy=0 0 0
- joint spine_0: origin xyz=0 0 0.15 rpy=0 0 0 -> xyz=0 0 0.0900777328402 rpy=0 0 0
