Commit message: Joystick ROS Test

File: urdf/test_arm_v2.urdf (robot description, URDF)
Before this commit: robot third_arm, 12 links, 11 joints
Links:
- link block_to_base: geometry visual cylinder length=0.1 radius=0.11

Commit message: IK Testing on random translations

File: urdf/test_arm_v2.urdf (robot description, URDF)
Before this commit: robot third_arm, 12 links, 11 joints
Joints:
- joint base_to_motor1: limit lower=-1.5708 upper=1.5708 effort=10 velocity=0.314 -> lower=-3.14 upper=3.14 effort=10 velocity=0.314

File: urdf/third_arm_5dof.urdf (robot description, URDF)
Before this commit: robot third_arm, 9 links, 8 joints
Links:
- added link environment_x; visual cylinder length=0.0 radius=0.0
- added link environment_y; visual cylinder length=0.0 radius=0.0
- added link environment_z; visual cylinder length=0.0 radius=0.0
- added link gripper_end_point; visual box size=.0 .0 .0
- link base_motor: geometry visual cylinder length=0.08 radius=0.05
- link extend_link2: geometry visual box size=0.07 .33 .07
- link wrist_plate: geometry visual box size=0.07 .035 .07
- link wrist_rotation_motor: geometry visual cylinder length=0.09 radius=0.03
Joints:
- added joint env_x: type prismatic, parent environment_x, child environment_y, origin xyz=0 0 0 rpy=0 0 0, axis 1 0 0, limit lower=-1 upper=1 effort=100 velocity=10
- added joint env_y: type prismatic, parent environment_y, child environment_z, origin xyz=0 0 0 rpy=0 0 0, axis 0 1 0, limit lower=-1 upper=1 effort=100 velocity=10
- added joint env_z_to_base: type prismatic, parent environment_z, child base_link, origin xyz=0 0 0 rpy=0 0 0, axis 0 0 1, limit lower=-1 upper=1 effort=100 velocity=10
- added joint gripper_end_point: type fixed, parent gripper_plate, child gripper_end_point, origin xyz=0.05 0 0 rpy=0 0 0
- joint base_to_motor1: limit lower=-1.5708 upper=1.5708 effort=10 velocity=0.314 -> lower=-3.14 upper=3.14 effort=10 velocity=0.314; origin xyz=0 0 0.00 rpy=0 0 -1.5708 -> xyz=0 0 0.0 rpy=0 0 0
- joint extension: origin xyz=0 0.125 0 rpy=0 0 0 -> xyz=0 0.1 0 rpy=0 0 0
- joint motor2_to_extend1: origin xyz=0 0.05 0 rpy=0 0 0 -> xyz=0 0.1 0 rpy=0 0 0
- joint swivel_to_motor2: origin xyz=0 0 -0.085 rpy=1.5708 3.14159 1.5708 -> xyz=0 0 -0.08 rpy=1.5708 3.14159 1.5708
- joint wrist_motor2_to_wrist_tilt_motor: origin xyz=0 0.065 0 rpy=0 0 -1.5708 -> xyz=0 0.045 0 rpy=0 0 -1.5708
- joint wrist_motor_to_extension: origin xyz=0 0.13 0 rpy=0 0 0 -> xyz=0 0.165 0 rpy=0 0 0
- joint wrist_plate_to_gripper_plate: origin xyz=0 0.1 0 rpy=1.5708 0 1.5708 -> xyz=0 0.0675 0 rpy=1.5708 0 1.5708
- joint wrist_tilt_motor_to_plate: origin xyz=0 0.035 0 rpy=0 0 0 -> xyz=0 0.0175 0 rpy=0 0 0

File: urdf/third_arm_6dof.urdf (robot description, URDF)
Before this commit: robot third_arm, 11 links, 10 joints
Links:
- added link finger1, mass 1; visual box size=0.01 .1 .02
- added link finger2, mass 1; visual box size=0.01 .1 .02
Joints:
- added joint finger1_to_gripper_motor: type revolute, parent gripper_motor, child finger1, origin xyz=0 0 0 rpy=0 0 0, axis 0 0 1, limit lower=0 upper=1 effort=5 velocity=0.5
- added joint finger2_to_gripper_motor: type revolute, parent gripper_motor, child finger2, origin xyz=0 0 0 rpy=0 0 0, axis 0 0 1, limit lower=-1 upper=0 effort=5 velocity=0.5, mimic joint=finger1_to_gripper_motor multiplier=-1

File: urdf/third_arm_kevin.urdf (robot description, URDF)
Before this commit: robot third_arm, 9 links, 8 joints
Links:
- added link finger1, mass 1; visual box size=0.01 .1 .02
- added link finger2, mass 1; visual box size=0.01 .1 .02
Joints:
- added joint finger1_to_gripper_motor: type revolute, parent gripper_motor, child finger1, origin xyz=0 0 0 rpy=0 0 0, axis 0 0 1, limit lower=0 upper=1 effort=5 velocity=0.5
- added joint finger2_to_gripper_motor: type revolute, parent gripper_motor, child finger2, origin xyz=0 0 0 rpy=0 0 0, axis 0 0 1, limit lower=-1 upper=0 effort=5 velocity=0.5, mimic joint=finger1_to_gripper_motor multiplier=-1
