Commit message: 6dof Joystick

File: urdf/third_arm_5dof.urdf (robot description, URDF)
Before this commit: robot third_arm, 9 links, 8 joints
Links:
- added link wrist_motor2, mass 1; visual cylinder length=0.05 radius=0.03
- added link wrist_motor3, mass 1; visual cylinder length=0.05 radius=0.03
Joints:
- added joint wrist_motor2_to_wrist_motor3: type revolute, parent wrist_motor2, child wrist_motor3, origin xyz=0 0.05 0 rpy=0 0 0, axis 0 0 1, limit lower=-1.5708 upper=1.5708 effort=5 velocity=0.5
- added joint wrist_motor_to_wrist_motor2: type revolute, parent wrist_motor, child wrist_motor2, origin xyz=0 0.05 0 rpy=0 0 0, axis 0 1 0, limit lower=-1.5708 upper=1.5708 effort=5 velocity=0.5
- joint wrist_motor2_to_wrist_tilt_motor: parent wrist_motor -> wrist_motor3

File: urdf/third_arm_6dof.urdf (robot description, URDF)
Before this commit: robot third_arm, 9 links, 8 joints
Links:
- added link wrist_motor2, mass 1; visual cylinder length=0.05 radius=0.03
- added link wrist_motor3, mass 1; visual cylinder length=0.05 radius=0.03
Joints:
- removed joint wrist_motor2_to_wrist_tilt_motor
- added joint wrist_motor2_to_wrist_motor3: type revolute, parent wrist_motor2, child wrist_motor3, origin xyz=0 0.06 0 rpy=0 0 0, axis 0 0 1, limit lower=-1.5708 upper=1.5708 effort=5 velocity=0.5
- added joint wrist_motor3_to_wrist_tilt_motor: type revolute, parent wrist_motor3, child wrist_tilt_motor, origin xyz=0 0.06 0 rpy=0 0 0, axis 1 0 0, limit lower=-1.5708 upper=1.5708 effort=5 velocity=0.5
- added joint wrist_motor_to_wrist_motor2: type revolute, parent wrist_motor, child wrist_motor2, origin xyz=0 0.05 0 rpy=0 0 0, axis 0 1 0, limit lower=-1.5708 upper=1.5708 effort=5 velocity=0.5

Commit message: added IK moveIt support

File: urdf/third_arm_5dof.urdf (robot description, URDF)
Before this commit: robot third_arm, 11 links, 10 joints
Links:
- removed link gripper_motor
- removed link wrist_motor
- removed link wrist_motor2
- removed link wrist_motor3
- added link gripper_plate; visual box size=.1 .03 .03
- added link wrist_rotation_motor, mass 1; visual cylinder length=0.06 radius=0.03
- link base_link: geometry visual cylinder length=0.05 radius=0.05
- link base_motor: geometry visual cylinder length=0.05 radius=0.05
- link lift_motor: geometry visual cylinder length=0.1 radius=0.05
Joints:
- removed joint gripper_motor_to_plate
- removed joint wrist_motor2_to_wrist_motor3
- removed joint wrist_motor_to_wrist_motor2
- added joint wrist_plate_to_gripper_plate: type fixed, parent wrist_plate, child gripper_plate, origin xyz=0 0.1 0 rpy=1.5708 0 1.5708
- joint base_to_motor1: origin xyz=0 0 -0.1 rpy=0 0 0 -> xyz=0 0 0.00 rpy=0 0 -1.5708
- joint extension: axis (none) -> 0 1 0; limit (none) -> lower=0 upper=0.12 effort=10 velocity=5; type fixed -> prismatic
- joint swivel_to_motor2: limit lower=-1.5708 upper=1.5708 effort=10 velocity=0.314 -> lower=0 upper=1.5708 effort=10 velocity=0.314; origin xyz=0 0.16 0 rpy=1.5708 1.5708 1.5708 -> xyz=0 0 -0.085 rpy=1.5708 3.14159 1.5708
- joint wrist_motor2_to_wrist_tilt_motor: axis 1 0 0 -> 0 0 1; limit lower=-1.5708 upper=1.5708 effort=5 velocity=0.5 -> lower=0 upper=3.14159 effort=5 velocity=0.5; origin xyz=0 0.06 0 rpy=0 0 0 -> xyz=0 0.065 0 rpy=0 0 -1.5708; parent wrist_motor3 -> wrist_rotation_motor
- joint wrist_motor_to_extension: child wrist_motor -> wrist_rotation_motor; origin xyz=0 0.125 0 rpy=0 0 0 -> xyz=0 0.13 0 rpy=0 0 0

Commit message: Somewhat success in hold

File: urdf/third_arm_5dof.urdf (robot description, URDF)
Before this commit: robot third_arm, 13 links, 12 joints
Joints:
- removed joint base_to_motor1
- removed joint extension
- removed joint swivel_to_motor2
- removed joint wrist_motor2_to_wrist_tilt_motor
- removed joint wrist_motor_to_extension
- added joint horizontal_panning: type revolute, parent base_link, child base_motor, origin xyz=0 0 0.0 rpy=0 0 -1.5708, axis 0 0 1, limit lower=-3.14 upper=3.14 effort=10 velocity=3.14
- added joint length_extension: type prismatic, parent extend_link1, child extend_link2, origin xyz=0 0.065 0 rpy=0 0 0, axis 0 1 0, limit lower=0 upper=0.12 effort=10 velocity=5
- added joint vertical_pitching: type revolute, parent base_motor, child lift_motor, origin xyz=0 0 -0.08 rpy=1.5708 3.14159 1.5708, axis 0 0 1, limit lower=0 upper=1.5708 effort=10 velocity=0.314
- added joint wrist_pitching: type revolute, parent wrist_rotation_motor, child wrist_tilt_motor, origin xyz=0 0.045 0 rpy=0 0 -1.5708, axis 0 0 1, limit lower=0 upper=3.14159 effort=5 velocity=0.5
- added joint wrist_rotation: type revolute, parent extend_link2, child wrist_rotation_motor, origin xyz=0 0.165 0 rpy=0 0 0, axis 0 1 0, limit lower=-3.14 upper=3.14 effort=5 velocity=0.5

Commit message: added launch file and updated urdf to load passive robot into gazebo, no actuators/controls yet

File: urdf/third_arm_5dof.urdf (robot description, URDF)
Before this commit: robot third_arm, 13 links, 12 joints
Links:
- link environment_x: mass None -> 1.0; geometry collision cylinder length=0.0 radius=0.0; visual cylinder length=0.0 radius=0.0
