Commit message: added a dummy base link so that the robot is fixed to the world in gazebo

File: urdf/third_arm_gazebo.urdf (robot description, URDF)
Before this commit: robot wrta, 13 links, 12 joints
Links:
- added link world
Joints:
- added joint fixed: type fixed, parent world, child environment_x
