Commit message: changed the base/env links to be fixed for gazebo urdf, to prevent the connection point sliding. reduced the moments of inertia. set the motor link mass to correspond to the corresponding dynamixel motors, reduced the mass of the other links to equally sum up to 2kg, to correspond to the published specs. obviously this is an estimate. Also reduced the base pan and lift motorlimits to 6 Nm

File: urdf/wrta_gazebo.urdf (robot description, URDF)
Before this commit: robot wrta, 14 links, 13 joints
Links:
- link base_link: mass 1.0 -> 0.2
- link base_motor: mass 1 -> 0.135
- link extend_link1: mass 1 -> 0.077
- link extend_link2: mass 1 -> 0.2
- link gripper_end_point: mass 1 -> 0.2
- link gripper_plate: mass 1 -> 0.2
- link lift_motor: mass 1 -> 0.135
- link wrist_plate: mass 1 -> 0.2
- link wrist_rotation_motor: mass 1 -> 0.0546
- link wrist_tilt_motor: mass 1 -> 0.0546
Joints:
- joint env_x: limit lower=-1 upper=1 effort=100 velocity=10 -> (none); type prismatic -> fixed
- joint env_y: limit lower=-1 upper=1 effort=100 velocity=10 -> (none); origin xyz=0 0 0 rpy=0 0 0 -> xyz=0 0 2 rpy=0 0 0; type prismatic -> fixed
- joint env_z_to_base: limit lower=-1 upper=1 effort=100 velocity=10 -> (none); type prismatic -> fixed
- joint horizontal_panning: limit lower=-3.14 upper=3.14 effort=10 velocity=3.14 -> lower=-3.14 upper=3.14 effort=6 velocity=3.14
- joint vertical_pitching: limit lower=0 upper=1.5708 effort=10 velocity=0.314 -> lower=0 upper=1.5708 effort=6 velocity=0.314
